Commit message: Replace robot.urdf file to make spheres black

File: urdf/robot.urdf (robot description, URDF)
Before this commit: robot myrobot, 9 links, 8 joints
Links:
- link sphere0: geometry collision sphere radius=0.5; visual sphere radius=0.5
- link sphere1: geometry collision sphere radius=0.3; visual sphere radius=0.3
- link sphere_base: geometry collision sphere radius=0.5; visual sphere radius=0.5
